File: hardware/kicad/atlastag.kicad_sch (KiCad schematic)
At the start: 0 parts

Commit message: fix(hardware): audit PR #4, implement complete baseboard schematic, and reconcile status claims
- Capture complete KiCad 10 baseboard schematic with real symbols, nets, power ports, and verified footprints
- Decouple Cellular/GNSS modem via 16-pin modular mezzanine interface to keep platform decision open
- Add Microchip MCP73831 212 mA linear charger, AP2112K-3.3 LDO, Winbond W25Q32 SOIC-8 flash, Nano-SIM socket, and motion breakout header
- Run schematic ERC and commit authoritative report (hardware/kicad/atlastag_erc.rpt)
- Clarify firmware/src/main.c as an architectural stub using simulated ADC values
- Reconcile BOMs at verified INR rate (₹96.70/USD) distinguishing .70 baseboard build from .25 total system projection
- Mark gerbers as strictly NOT FOR FABRICATION pending interactive GUI routing and DRC
- Update README.md with comprehensive architecture, operating cycle, and Concept & Vision Reel callouts
Parts:
- added C1: 10uF VBUS, Capacitor_SMD:C_0603_1608Metric, symbol Device:C
- added C2: 10uF VBAT, Capacitor_SMD:C_0603_1608Metric, symbol Device:C
- added C3: 100uF Bulk, Capacitor_Tantalum_SMD:CP_EIA-3528-21_Kemet-B_HandSolder, symbol Device:C_Polarized
- added C4: 10nF ADC, Capacitor_SMD:C_0603_1608Metric, symbol Device:C
- added C5: 4.7uF LDO_IN, Capacitor_SMD:C_0603_1608Metric, symbol Device:C
- added C6: 4.7uF LDO_OUT, Capacitor_SMD:C_0603_1608Metric, symbol Device:C
- added C7: 100nF Flash, Capacitor_SMD:C_0603_1608Metric, symbol Device:C
- added C8: 4.7uF Flash, Capacitor_SMD:C_0603_1608Metric, symbol Device:C
- added D1: Red CHG, LED_SMD:LED_0603_1608Metric, symbol Device:LED
- added D2: Green 3V3, LED_SMD:LED_0603_1608Metric, symbol Device:LED
- added J1: USB-C 5V In, Connector_USB:USB_C_Receptacle_HRO_TYPE-C-31-M-12, symbol Connector:USB_C_Receptacle_USB2.0_16P
- added J2: Li-Po Battery, Connector_JST:JST_PH_S2B-PH-K_1x02_P2.00mm_Horizontal, symbol Connector_Generic:Conn_01x02
- added J3: Motion Port, Connector_PinHeader_2.54mm:PinHeader_1x05_P2.54mm_Vertical, symbol Connector_Generic:Conn_01x05
- added J4: Modem Mezzanine, Connector_PinHeader_2.54mm:PinHeader_2x08_P2.54mm_Vertical, symbol Connector_Generic:Conn_02x08_Odd_Even
- added J5: Nano-SIM, Connector_Card:nanoSIM_GCT_SIM8060-6-0-14-00, symbol Connector:SIM_Card_Shielded
- added R1: 5.1k CC1, Resistor_SMD:R_0603_1608Metric, symbol Device:R
- added R10: 10k DATA_PU, Resistor_SMD:R_0603_1608Metric, symbol Device:R
- added R11: 100k BTN_PU, Resistor_SMD:R_0603_1608Metric, symbol Device:R
- added R12: 4.7k SCL_PU, Resistor_SMD:R_0603_1608Metric, symbol Device:R
- added R13: 4.7k SDA_PU, Resistor_SMD:R_0603_1608Metric, symbol Device:R
- added R14: 10k WP_PU, Resistor_SMD:R_0603_1608Metric, symbol Device:R
- added R15: 10k HOLD_PU, Resistor_SMD:R_0603_1608Metric, symbol Device:R
- added R2: 5.1k CC2, Resistor_SMD:R_0603_1608Metric, symbol Device:R
- added R3: 1.5k LED, Resistor_SMD:R_0603_1608Metric, symbol Device:R
- added R4: 4.7k PROG, Resistor_SMD:R_0603_1608Metric, symbol Device:R
- added R5: 1.0M DIV_HI, Resistor_SMD:R_0603_1608Metric, symbol Device:R
- added R6: 1.0M DIV_LO, Resistor_SMD:R_0603_1608Metric, symbol Device:R
- added R7: 100k EN, Resistor_SMD:R_0603_1608Metric, symbol Device:R
- added R8: 2.2k LED, Resistor_SMD:R_0603_1608Metric, symbol Device:R
- added R9: 10k CS_PU, Resistor_SMD:R_0603_1608Metric, symbol Device:R
- added SW1: User Button, Button_Switch_SMD:SW_SPST_PTS645Sx43SMTR92, symbol Switch:SW_Push
- added U1: MCP73831T-2ACI/OT, Package_TO_SOT_SMD:SOT-23-5, symbol Battery_Management:MCP73831-2-OT
- added U2: AP2112K-3.3, Package_TO_SOT_SMD:SOT-23-5, symbol Regulator_Linear:AP2112K-3.3
- added U3: W25Q32JVSSIQ, Package_SO:SOIC-8_5.3x5.3mm_P1.27mm, symbol Memory_Flash:W25Q32JVSS
Connections:
- new net: R3.2, U1.1 (STAT)
- new net: R4.1, U1.5 (PROG)
- new net: J1.A5 (CC1), R1.1
- new net: D2.1 (K), R8.1
- new net: R7.2, U2.3 (EN)
- new net +3V3: C6.1, C7.1, C8.1, D2.2 (A), J3.1 (Pin_1), J4.5 (Pin_5), R11.1, R12.1, R13.1, R14.1, R14.2, R15.1, R15.2, R9.1, U2.5 (VOUT), U3.3 (~{WP}/IO_{2}), U3.7 (~{HOLD}/~{RESET}/IO_{3}), U3.8 (VCC)
- new net FLASH_CS: R9.2, U3.1 (~{CS})
- new net GND: C1.2, C2.2, C3.2, C4.2, C5.2, C6.2, C7.2, C8.2, J1.A1 (GND), J1.A12 (GND), J1.B1 (GND), J1.B12 (GND), J1.B5 (CC2), J1.SH (SHIELD), J2.2 (Pin_2), J3.2 (Pin_2), J4.3 (Pin_3), J4.4 (Pin_4), J5.5 (GND), J5.SH, R1.2, R2.1, R2.2, R4.2, R6.2, R8.2, SW1.2, U1.2 (V_{SS}), U2.2 (GND), U3.4 (GND)
- new net I2C_SCL: J3.3 (Pin_3), R12.2
- new net I2C_SDA: J3.4 (Pin_4), R13.2
- new net MODEM_PWRKEY: J4.6 (Pin_6)
- new net MODEM_RESET: J4.7 (Pin_7)
- new net MODEM_STATUS: J4.8 (Pin_8)
- new net MOTION_INT: J3.5 (Pin_5)
- new net SIM_CLK: J4.15 (Pin_15), J5.3 (CLK)
- new net SIM_DATA: J4.16 (Pin_16), J5.7 (I/O), R10.2
- new net SIM_RST: J4.14 (Pin_14), J5.2 (RST)
- new net SIM_VCC: J4.13 (Pin_13), J5.1 (VCC), R10.1
- new net SPI_CLK: U3.6 (CLK)
- new net SPI_MISO: U3.2 (DO/IO_{1})
- new net SPI_MOSI: U3.5 (DI/IO_{0})
- new net UART_CTS: J4.12 (Pin_12)
- new net UART_RTS: J4.11 (Pin_11)
- new net UART_RX: J4.10 (Pin_10)
- new net UART_TX: J4.9 (Pin_9)
- new net USER_BTN: R11.2, SW1.1
- new net VBAT: C2.1, C3.1, C5.1, D1.1 (K), J2.1 (Pin_1), J4.1 (Pin_1), J4.2 (Pin_2), R3.1, R5.1, R7.1, U1.3 (V_{BAT}), U2.1 (VIN)
- new net VBAT_ADC: C4.1, R5.2, R6.1
- new net VBUS: C1.1, D1.2 (A), J1.A4 (VBUS), J1.A9 (VBUS), J1.B4 (VBUS), J1.B9 (VBUS), U1.4 (V_{DD})
- no-connect marks 0 -> 8
